Commit message: 真机模型弃减面改原始网格 + 加载进度条（用户决策：保真优先）
- visual/ = 官方 DM 原始分色网格 30 件 21MB；URDF 副本路径重写
- 删除 make_visual_lo.py 与 visual_lo 低模（视觉损失被否决）
- 加载覆盖层：说明 + 青色进度条 + 体积提示 + 失败态；完成渐隐
- 验证：30/30 mesh、进度条走完移除、动画在跑

File: web/public/models/ReBot_Arm_DM_preview.urdf (robot description, URDF)
Before this commit: robot ReBot_Arm_DM, 10 links, 9 joints
Links:
- link base_link: geometry collision mesh filename=../meshes/collision/base_link.STL; visual mesh filename=visual/colored_base_link_hardware_black.stl
- link end_link: geometry collision mesh filename=../meshes/collision/gripper_base.stl; visual mesh filename=visual/colored_gripper_base_hardware_black.stl
- link finger_left_link: geometry collision mesh filename=../meshes/collision/left_finger.stl; visual mesh filename=../meshes/shared/colored_left_finger_carriage_grey.stl
- link finger_right_link: geometry collision mesh filename=../meshes/collision/right_finger.stl; visual mesh filename=../meshes/shared/colored_right_finger_carriage_grey.stl
- link link1: geometry collision mesh filename=../meshes/collision/link1.STL; visual mesh filename=visual/colored_link1_anodized_grey.stl
- link link2: geometry collision mesh filename=../meshes/collision/link2.STL; visual mesh filename=visual/colored_link2_anodized_grey.stl
- link link3: geometry collision mesh filename=../meshes/collision/link3.STL; visual mesh filename=visual/colored_link3_anodized_grey.stl
- link link4: geometry collision mesh filename=../meshes/collision/link4.STL; visual mesh filename=visual/colored_link4_anodized_grey.stl
- link link5: geometry collision mesh filename=../meshes/collision/link5.STL; visual mesh filename=visual/colored_link5_anodized_grey.stl
- link link6: geometry collision mesh filename=../meshes/collision/link6.STL; visual mesh filename=visual/colored_link6_hardware_black.stl

Commit message: P5-A 伴生服务骨架：FastAPI 静态托管 + WS 桥 + 前端双模探测
- web/server/main.py：dist 双路径托管（根+Pages base 前缀）+ /api/health
  + /ws 桥 hub（web/pc 角色、广播、最新状态补发——P5-B~E 地基）
- src/companion.ts：探测模块（在线→实时模式，离线→演示模式）
- 总览页伴生服务卡接探测（实测转绿）；WS 三客户端广播/补发全链路实测
- 附带根治：preview.urdf shared 引用漏重写致 4 条 URDFLoader 404（多级
  相对路径被 urdf-loader 剥段）；URDF fetch 缓存坑加 ?v 破除——34/34 STL 全 200

File: web/public/models/ReBot_Arm_DM_preview.urdf (robot description, URDF)
Before this commit: robot ReBot_Arm_DM, 10 links, 9 joints
Links:
- link finger_left_link: geometry collision mesh filename=../meshes/collision/left_finger.stl; visual mesh filename=shared/colored_left_finger_carriage_grey.stl
- link finger_right_link: geometry collision mesh filename=../meshes/collision/right_finger.stl; visual mesh filename=shared/colored_right_finger_carriage_grey.stl

Commit message: 双代理全面审查落地：性能双杠杆 + 架构 P1 三项
- 性能杠杆 1：构建时 gzip（wasm/STL/urdf 全格式，实测压至 25-32%）
  + 前端 DecompressionStream 解压 + .gz 404 回退；sim/home 双页接入
- 性能杠杆 2：sim 页 WASM 与模型预取并行化（原严格串行）
- 删 URDF 10 个 collision 死引用（404 源+文案闪烁）
- 架构：sim.css 外迁（sim.html 235→46 行）；--font-mono 令牌收敛 11 处
  漂移栈；watchCompanion 统一三页探测（live 三块合并/home 换用）；
  .page-shell/.hud-card 原语；meta description 补全
- 实测：总览 gz 6.7MB（-69%）、sim gz 6.6MB 零 404、TCP 0.3mm 全站绿

File: web/public/models/ReBot_Arm_DM_preview.urdf (robot description, URDF)
Before this commit: robot ReBot_Arm_DM, 10 links, 9 joints
Links:
- link base_link: geometry visual mesh filename=visual/colored_base_link_hardware_black.stl; visual mesh filename=visual/colored_base_link_matte_black.stl
- link end_link: geometry visual mesh filename=visual/colored_gripper_base_hardware_black.stl; visual mesh filename=visual/colored_gripper_base_metal.stl
- link finger_left_link: geometry visual mesh filename=shared/colored_left_finger_carriage_grey.stl; visual mesh filename=shared/colored_left_finger_travel_stop_yellow.stl
- link finger_right_link: geometry visual mesh filename=shared/colored_right_finger_carriage_grey.stl; visual mesh filename=shared/colored_right_finger_travel_stop_yellow.stl
- link link1: geometry visual mesh filename=visual/colored_link1_anodized_grey.stl; visual mesh filename=visual/colored_link1_hardware_black.stl
- link link2: geometry visual mesh filename=visual/colored_link2_anodized_grey.stl; visual mesh filename=visual/colored_link2_hardware_black.stl
- link link3: geometry visual mesh filename=visual/colored_link3_anodized_grey.stl; visual mesh filename=visual/colored_link3_hardware_black.stl
- link link4: geometry visual mesh filename=visual/colored_link4_anodized_grey.stl; visual mesh filename=visual/colored_link4_hardware_black.stl
- link link5: geometry visual mesh filename=visual/colored_link5_anodized_grey.stl; visual mesh filename=visual/colored_link5_hardware_black.stl
- link link6: geometry visual mesh filename=visual/colored_link6_hardware_black.stl; visual mesh filename=visual/colored_link6_matte_black.stl
